File: pcb/Sensexpansion.kicad_sch (KiCad schematic)
At the start: 11 parts, among them U1 LIS3DH, U2 BME280

Commit message: stufs
Parts:
- C1, C2: LCSC Part # (none) -> C60474
- D1: LCSC Part # (none) -> C20608782
- R1: LCSC Part # (none) -> C140179
- R2: LCSC Part # (none) -> C140197
- R3: value R -> 300; LCSC Part # (none) -> C25102
- R4, R5: LCSC Part # (none) -> C140158
- U1: LCSC Part # (none) -> C15134
- U2: LCSC Part # (none) -> C92489
Other:
- note removed: "TODO: calculate needed resistance after picking led on lcsc"
Changed lines of the file:
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@@
 	(generator_version "10.0")
 	(paper "A4")
-	(text "TODO: calculate needed resistance after picking led on lcsc"
-		(exclude_from_sim no)
-		(at 188.468 76.962 0)
-		(effects
-			(font
-				(size 1.27 1.27)
-			)
-		)
-	)
 	(junction
 		(at 45.72 49.53)
@@
 			)
 		)
+		(property "LCSC Part #" "C140158"
+			(at 196.85 44.45 0)
+			(hide yes)
+			(show_name no)
+			(do_not_autoplace no)
+			(effects
+				(font
+					(size 1.27 1.27)
+				)
+			)
+		)
 		(pin "1"
 		)
@@
 			)
 		)
+		(property "LCSC Part #" "C15134"
+			(at 66.04 49.53 0)
+			(hide yes)
+			(show_name no)
+			(do_not_autoplace no)
+			(effects
+				(font
+					(size 1.27 1.27)
+				)
+			)
+		)
 		(pin "12"
 		)
@@
 			)
 		)
+		(property "LCSC Part #" "C92489"
+			(at 104.14 52.07 0)
+			(hide yes)
+			(show_name no)
+			(do_not_autoplace no)
+			(effects
+				(font
+					(size 1.27 1.27)
+				)
+			)
+		)
 		(pin "3"
 		)
@@
 			)
 		)
+		(property "LCSC Part #" "C20608782"
+			(at 154.94 81.28 0)
+			(hide yes)
+			(show_name no)
+			(do_not_autoplace no)
+			(effects
+				(font
+					(size 1.27 1.27)
+				)
+			)
+		)
 		(pin "1"
 		)
@@
 			)
 		)
-		(property "Value" "R"
+		(property "Value" "300"
 			(at 157.48 73.6599 0)
 			(show_name no)
@@
 		)
 		(property "Description" "Resistor"
+			(at 154.94 72.39 0)
+			(hide yes)
+			(show_name no)
+			(do_not_autoplace no)
+			(effects
+				(font
+					(size 1.27 1.27)
+				)
+			)
+		)
+		(property "LCSC Part #" "C25102"
 			(at 154.94 72.39 0)
 			(hide yes)
@@
 			)
 		)
+		(property "LCSC Part #" "C140197"
+			(at 149.86 53.34 0)
+			(hide yes)
+			(show_name no)
+			(do_not_autoplace no)
+			(effects
+				(font
+					(size 1.27 1.27)
+				)
+			)
+		)
 		(pin "1"
 		)
@@
 			)
 		)
+		(property "LCSC Part #" "C60474"
+			(at 88.9 39.37 0)
+			(hide yes)
+			(show_name no)
+			(do_not_autoplace no)
+			(effects
+				(font
+					(size 1.27 1.27)
+				)
+			)
+		)
 		(pin "2"
 		)
@@
 			)
 		)
+		(property "LCSC Part #" "C140158"
+			(at 187.96 41.91 0)
+			(hide yes)
+			(show_name no)
+			(do_not_autoplace no)
+			(effects
+				(font
+					(size 1.27 1.27)
+				)
+			)
+		)
 		(pin "1"
 		)
@@
 			)
 		)
+		(property "LCSC Part #" "C140179"
+			(at 142.24 50.8 0)
+			(hide yes)
+			(show_name no)
+			(do_not_autoplace no)
+			(effects
+				(font
+					(size 1.27 1.27)
+				)
+			)
+		)
 		(pin "1"
 		)
@@
 			(at 85.09 39.37 0)
 			(hide yes)
+			(show_name no)
+			(do_not_autoplace no)
+			(effects
+				(font
+					(size 1.27 1.27)
+				)
+			)
+		)
+		(property "LCSC Part #" "C60474"
+			(at 85.09 39.37 0)
+			(hide yes)
